File: kicad/WiredSEK.sch (KiCad schematic (older format))
At the start: 55 parts, among them J1 Conn_01x34, J2 USB_B_Micro, J3 AVR-JTAG-10, J4 Serial RX/TX, J5 Testpad, SW1 HWB_SW, SW2 RST_SW, U1 USBLC6-2SC6, U2 AT90USB646-AU, Y1 16 Mhz

Commit message: JLCPCB Order REV 1
Parts:
- C2: LCSC (none) -> C15850; LCSC Part # C15850 -> (none)
- C3, C4: LCSC (none) -> C1647; LCSC Part # C1647 -> (none)
- C5: LCSC (none) -> C15849; LCSC Part # C15849 -> (none)
- C6, C7, C8, C9: LCSC (none) -> C57112; LCSC Part # C57112 -> (none)
- D1: LCSC (none) -> C72041; LCSC Part # C72041 -> (none)
- D2: LCSC (none) -> C72043; LCSC Part # C72043 -> (none)
- F1: LCSC (none) -> C369159; LCSC Part # C369159 -> (none)
- R1, R2: LCSC (none) -> C17414; LCSC Part # C17414 -> (none)
- R10, R11, R12, R3, R4, R9: LCSC (none) -> C17710; LCSC Part # C17710 -> (none)
- R5, R6: LCSC (none) -> C25295; LCSC Part # C25295 -> (none)
- R7: value ?? -> 10k; LCSC (none) -> C17414
- R8: value ?? -> 2k; LCSC (none) -> C17710
- SW1, SW2: LCSC (none) -> C115357; LCSC Part # C115357 -> (none)
- U1: LCSC (none) -> C558442; LCSC Part # C558442 -> (none)
- Y1: LCSC (none) -> C13738; LCSC Part # X1E000021011900 -> (none)
Changed lines of the file:
@@
 F 2 "Package_TO_SOT_SMD:SOT-23-6" H 1900 2850 50  0001 C CNN
 F 3 "https://www.st.com/resource/en/datasheet/usblc6-2.pdf" H 2100 3700 50  0001 C CNN
-F 4 "C558442" H 1900 3350 50  0001 C CNN "LCSC Part #"
+F 4 "C558442" H 1900 3350 50  0001 C CNN "LCSC"
 	1    1900 3350
 	1    0    0    -1
@@
 F 2 "Resistor_SMD:R_0805_2012Metric_Pad1.20x1.40mm_HandSolder" H 6000 2450 50  0001 C CNN
 F 3 "~" H 6000 2450 50  0001 C CNN
-F 4 "C25295" H 6000 2450 50  0001 C CNN "LCSC Part #"
+F 4 "C25295" H 6000 2450 50  0001 C CNN "LCSC"
 	1    6000 2450
 	0    1    1    0
@@
 F 2 "Resistor_SMD:R_0805_2012Metric_Pad1.20x1.40mm_HandSolder" H 6000 2550 50  0001 C CNN
 F 3 "~" H 6000 2550 50  0001 C CNN
-F 4 "C25295" H 6000 2550 50  0001 C CNN "LCSC Part #"
+F 4 "C25295" H 6000 2550 50  0001 C CNN "LCSC"
 	1    6000 2550
 	0    1    1    0
@@
 F 2 "Capacitor_SMD:C_0603_1608Metric_Pad1.08x0.95mm_HandSolder" H 8650 950 50  0001 C CNN
 F 3 "~" H 8650 950 50  0001 C CNN
-F 4 "C57112" H 8650 950 50  0001 C CNN "LCSC Part #"
+F 4 "C57112" H 8650 950 50  0001 C CNN "LCSC"
 	1    8650 950
 	1    0    0    -1
@@
 F 2 "Capacitor_SMD:C_0603_1608Metric_Pad1.08x0.95mm_HandSolder" H 8900 950 50  0001 C CNN
 F 3 "~" H 8900 950 50  0001 C CNN
-F 4 "C57112" H 8900 950 50  0001 C CNN "LCSC Part #"
+F 4 "C57112" H 8900 950 50  0001 C CNN "LCSC"
 	1    8900 950
 	1    0    0    -1
@@
 F 2 "Capacitor_SMD:C_0603_1608Metric_Pad1.08x0.95mm_HandSolder" H 9150 950 50  0001 C CNN
 F 3 "~" H 9150 950 50  0001 C CNN
-F 4 "C57112" H 9150 950 50  0001 C CNN "LCSC Part #"
+F 4 "C57112" H 9150 950 50  0001 C CNN "LCSC"
 	1    9150 950
 	1    0    0    -1
@@
 F 2 "Capacitor_SMD:C_0603_1608Metric_Pad1.08x0.95mm_HandSolder" H 6100 3150 50  0001 C CNN
 F 3 "~" H 6100 3150 50  0001 C CNN
-F 4 "C15849" H 6100 3150 50  0001 C CNN "LCSC Part #"
+F 4 "C15849" H 6100 3150 50  0001 C CNN "LCSC"
 	1    6100 3150
 	1    0    0    -1
@@
 F 2 "Capacitor_SMD:C_0805_2012Metric_Pad1.18x1.45mm_HandSolder" H 4250 1100 50  0001 C CNN
 F 3 "~" H 4250 1100 50  0001 C CNN
-F 4 "C15850" H 4250 1100 50  0001 C CNN "LCSC Part #"
+F 4 "C15850" H 4250 1100 50  0001 C CNN "LCSC"
 	1    4250 1100
 	1    0    0    -1
@@
 F 2 "Crystal:Crystal_SMD_3225-4Pin_3.2x2.5mm_HandSoldering" H 5550 5600 50  0001 C CNN
 F 3 "~" H 5550 5600 50  0001 C CNN
-F 4 "X1E000021011900" H 5550 5600 50  0001 C CNN "LCSC Part #"
+F 4 "C13738" H 5550 5600 50  0001 C CNN "LCSC"
 	1    5550 5600
 	0    1    1    0
@@
 F 2 "Capacitor_SMD:C_0603_1608Metric_Pad1.08x0.95mm_HandSolder" H 4850 5500 50  0001 C CNN
 F 3 "~" H 4850 5500 50  0001 C CNN
-F 4 "C1647" H 4850 5500 50  0001 C CNN "LCSC Part #"
+F 4 "C1647" H 4850 5500 50  0001 C CNN "LCSC"
 	1    4850 5500
 	0    1    1    0
@@
 F 2 "Capacitor_SMD:C_0603_1608Metric_Pad1.08x0.95mm_HandSolder" H 4850 5700 50  0001 C CNN
 F 3 "~" H 4850 5700 50  0001 C CNN
-F 4 "C1647" H 4850 5700 50  0001 C CNN "LCSC Part #"
+F 4 "C1647" H 4850 5700 50  0001 C CNN "LCSC"
 	1    4850 5700
 	0    1    1    0
@@
 F 2 "Resistor_SMD:R_0805_2012Metric_Pad1.20x1.40mm_HandSolder" H 2350 5300 50  0001 C CNN
 F 3 "~" H 2350 5300 50  0001 C CNN
-F 4 "C17414" H 2350 5300 50  0001 C CNN "LCSC Part #"
+F 4 "C17414" H 2350 5300 50  0001 C CNN "LCSC"
 	1    2350 5300
 	1    0    0    -1
@@
 F 2 "WiredSEK:SKRKAEE020" H 2350 6000 50  0001 C CNN
 F 3 "~" H 2350 6000 50  0001 C CNN
-F 4 "C115357" H 2350 5800 50  0001 C CNN "LCSC Part #"
+F 4 "C115357" H 2350 5800 50  0001 C CNN "LCSC"
 	1    2350 5800
 	0    1    1    0
@@
 F 2 "Fuse:Fuse_1206_3216Metric_Pad1.42x1.75mm_HandSolder" H 2500 1050 50  0001 C CNN
 F 3 "~" H 2500 1050 50  0001 C CNN
-F 4 "C369159" H 2500 1050 50  0001 C CNN "LCSC Part #"
+F 4 "C369159" H 2500 1050 50  0001 C CNN "LCSC"
 	1    2500 1050
 	1    0    0    -1
@@
 F 2 "Resistor_SMD:R_0805_2012Metric_Pad1.20x1.40mm_HandSolder" H 1000 5250 50  0001 C CNN
 F 3 "~" H 1000 5250 50  0001 C CNN
-F 4 "C17414" H 1000 5250 50  0001 C CNN "LCSC Part #"
+F 4 "C17414" H 1000 5250 50  0001 C CNN "LCSC"
 	1    1000 5250
 	1    0    0    -1
@@
 F 2 "WiredSEK:SKRKAEE020" H 1000 5950 50  0001 C CNN
 F 3 "~" H 1000 5950 50  0001 C CNN
-F 4 "C115357" H 1000 5750 50  0001 C CNN "LCSC Part #"
+F 4 "C115357" H 1000 5750 50  0001 C CNN "LCSC"
 	1    1000 5750
 	0    1    1    0
@@
 F 2 "LED_SMD:LED_0603_1608Metric_Pad1.05x0.95mm_HandSolder" V 3400 5450 50  0001 C CNN
 F 3 "~" V 3400 5450 50  0001 C CNN
-F 4 "C72041" H 3400 5450 50  0001 C CNN "LCSC Part #"
+F 4 "C72041" H 3400 5450 50  0001 C CNN "LCSC"
 	1    3400 5450
 	0    -1   -1   0
@@
 F 2 "Resistor_SMD:R_0805_2012Metric_Pad1.20x1.40mm_HandSolder" H 3400 5800 50  0001 C CNN
 F 3 "~" H 3400 5800 50  0001 C CNN
-F 4 "C17710" H 3400 5800 50  0001 C CNN "LCSC Part #"
+F 4 "C17710" H 3400 5800 50  0001 C CNN "LCSC"
 	1    3400 5800
 	1    0    0    -1
@@
 F 2 "LED_SMD:LED_0603_1608Metric_Pad1.05x0.95mm_HandSolder" V 4750 1100 50  0001 C CNN
 F 3 "~" V 4750 1100 50  0001 C CNN
-F 4 "C72043" H 4750 1100 50  0001 C CNN "LCSC Part #"
+F 4 "C72043" H 4750 1100 50  0001 C CNN "LCSC"
 	1    4750 1100
 	0    -1   -1   0
@@
 F 2 "Resistor_SMD:R_0805_2012Metric_Pad1.20x1.40mm_HandSolder" H 4750 1450 50  0001 C CNN
 F 3 "~" H 4750 1450 50  0001 C CNN
-F 4 "C17710" H 4750 1450 50  0001 C CNN "LCSC Part #"
+F 4 "C17710" H 4750 1450 50  0001 C CNN "LCSC"
 	1    4750 1450
 	1    0    0    -1
@@
 F 2 "Capacitor_SMD:C_0603_1608Metric_Pad1.08x0.95mm_HandSolder" H 9400 950 50  0001 C CNN
 F 3 "~" H 9400 950 50  0001 C CNN
-F 4 "C57112" H 9400 950 50  0001 C CNN "LCSC Part #"
+F 4 "C57112" H 9400 950 50  0001 C CNN "LCSC"
 	1    9400 950
 	1    0    0    -1
@@
 F 2 "Resistor_SMD:R_0805_2012Metric_Pad1.20x1.40mm_HandSolder" H 9700 5050 50  0001 C CNN
 F 3 "~" H 9700 5050 50  0001 C CNN
-F 4 "C17710" H 9700 5050 50  0001 C CNN "LCSC Part #"
+F 4 "C17710" H 9700 5050 50  0001 C CNN "LCSC"
 	1    9700 5050
 	1    0    0    -1
@@
 F 2 "Resistor_SMD:R_0805_2012Metric_Pad1.20x1.40mm_HandSolder" H 9600 5050 50  0001 C CNN
 F 3 "~" H 9600 5050 50  0001 C CNN
-F 4 "C17710" H 9600 5050 50  0001 C CNN "LCSC Part #"
+F 4 "C17710" H 9600 5050 50  0001 C CNN "LCSC"
 	1    9600 5050
 	1    0    0    -1
@@
 F 2 "Resistor_SMD:R_0805_2012Metric_Pad1.20x1.40mm_HandSolder" H 9450 2300 50  0001 C CNN
 F 3 "~" H 9450 2300 50  0001 C CNN
-F 4 "C17710" H 9450 2300 50  0001 C CNN "LCSC Part #"
+F 4 "C17710" H 9450 2300 50  0001 C CNN "LCSC"
 	1    9450 2300
 	-1   0    0    1
@@
 F 2 "Resistor_SMD:R_0805_2012Metric_Pad1.20x1.40mm_HandSolder" H 9550 2300 50  0001 C CNN
 F 3 "~" H 9550 2300 50  0001 C CNN
-F 4 "C17710" H 9550 2300 50  0001 C CNN "LCSC Part #"
+F 4 "C17710" H 9550 2300 50  0001 C CNN "LCSC"
 	1    9550 2300
 	-1   0    0    1
@@
 P 9350 2950
 F 0 "R7" H 9200 3000 50  0000 L CNN
-F 1 "??" H 9200 2900 50  0000 L CNN
+F 1 "10k" H 9200 2900 50  0000 L CNN
 F 2 "Resistor_SMD:R_0805_2012Metric_Pad1.20x1.40mm_HandSolder" H 9350 2950 50  0001 C CNN
 F 3 "~" H 9350 2950 50  0001 C CNN
-F 4 "" H 9350 2950 50  0001 C CNN "LCSC Part #"
+F 4 "C17414" H 9350 2950 50  0001 C CNN "LCSC"
 	1    9350 2950
 	1    0    0    -1
@@
 P 9450 2950
 F 0 "R8" H 9500 3000 50  0000 L CNN
-F 1 "??" H 9500 2900 50  0000 L CNN
+F 1 "2k" H 9500 2900 50  0000 L CNN
 F 2 "Resistor_SMD:R_0805_2012Metric_Pad1.20x1.40mm_HandSolder" H 9450 2950 50  0001 C CNN
 F 3 "~" H 9450 2950 50  0001 C CNN
-F 4 "" H 9450 2950 50  0001 C CNN "LCSC Part #"
+F 4 "C17710" H 9450 2950 50  0001 C CNN "LCSC"
 	1    9450 2950
 	1    0    0    -1
